Commit message: Refactor UVSMapServer and related files to improve world loading and model definitions

File: src/uvs_mapserver/models/agent.xacro (robot description, xacro)
@@ -3,5 +3,5 @@
         <xacro:if value="${vertex}">
             <xacro:property name="v" value="${vertex.pop(0)}"/>
-            <vertex>${v}</vertex>
+            <vertex x="${v[0]}" y="${v[1]}" />
             <xacro:unfoldVertex/>
         </xacro:if>
@@ -10,12 +10,11 @@
         <xacro:if value="${anchor}">
             <xacro:property name="a" value="${anchor.pop(0)}"/>
-            <anchor>${a}</anchor>
+            <anchor x="${a[0]}" y="${a[1]}" />
             <xacro:unfoldAnchor/>
         </xacro:if>
     </xacro:macro>
-    <xacro:macro name="defineAgent" params="name vertex:=^ anchor:=^ initpose:=${[0,0,0]}">
-        <agent>
-            <name>${name}</name>
-            <pose>${initpose}</pose>
+    <xacro:macro name="defineAgent" params="name vertex:=^ anchor:=^ initpose:=${[0,0,0]} limit_speed">
+        <agent name="${name}" max_speed="${limit_speed[0]}" min_speed="${limit_speed[1]}" max_angular_speed="${limit_speed[2]}" min_angular_speed="${limit_speed[3]}">
+            <pose x="${initpose[0]}" y="${initpose[1]}" theta="${initpose[2]}" />
             <xacro:unfoldVertex vertex="${list(vertex)}" />
             <xacro:unfoldAnchor anchor="${list(anchor)}" />

File: src/uvs_mapserver/models/cargo.xacro (robot description, xacro)
@@ -3,5 +3,5 @@
         <xacro:if value="${vertex}">
             <xacro:property name="v" value="${vertex.pop(0)}"/>
-            <vertex>${v}</vertex>
+            <vertex x="${v[0]}" y="${v[1]}" />
             <xacro:unfoldVertex/>
         </xacro:if>
@@ -10,15 +10,14 @@
         <xacro:if value="${anchor}">
             <xacro:property name="a" value="${anchor.pop(0)}"/>
-            <anchor>${a}</anchor>
+            <anchor x="${a[0]}" y="${a[1]}" />
             <xacro:unfoldAnchor/>
         </xacro:if>
     </xacro:macro>
     <xacro:macro name="defineCargo" params="name vertex:=^ anchor:=^ initpose:=${[0,0,0]}">
-        <Cargo>
-            <name>${name}</name>
-            <pose>${initpose}</pose>
+        <cargo name="${name}">
+            <pose x="${initpose[0]}" y="${initpose[1]}" theta="${initpose[2]}" />
             <xacro:unfoldVertex vertex="${list(vertex)}" />
             <xacro:unfoldAnchor anchor="${list(anchor)}" />
-        </Cargo>
+        </cargo>
     </xacro:macro>
 </world>

File: src/uvs_mapserver/models/ground.xacro (robot description, xacro)
@@ -3,5 +3,5 @@
         <xacro:if value="${vertex}">
             <xacro:property name="v" value="${vertex.pop(0)}"/>
-            <vertex>${v}</vertex>
+            <vertex x="${v[0]}" y="${v[1]}" />
             <xacro:unfoldVertex/>
         </xacro:if>
@@ -9,5 +9,5 @@
     <xacro:macro name="defineGround" params="vertex:=^ origin:=${[0,0]}">
         <ground>
-            <origin>${origin}</origin>
+            <origin x="${origin[0]}" y="${origin[1]}" />
             <xacro:unfoldVertex vertex="${list(vertex)}" />
         </ground>

File: src/uvs_mapserver/models/obstacle.xacro (robot description, xacro)
@@ -3,5 +3,5 @@
         <xacro:if value="${vertex}">
             <xacro:property name="v" value="${vertex.pop(0)}"/>
-            <vertex>${v}</vertex>
+            <vertex x="${v[0]}" y="${v[1]}" />
             <xacro:unfoldVertex/>
         </xacro:if>
@@ -9,5 +9,5 @@
     <xacro:macro name="defineObstacle" params="vertex:=^ pose:=${[0,0,0]}">
         <obstacle>
-            <pose>${pose}</pose>
+            <pose x="${pose[0]}" y="${pose[1]}" theta="${pose[2]}" />
             <xacro:unfoldVertex vertex="${list(vertex)}" />
         </obstacle>

File: src/uvs_mapserver/world/jxl3028.world.xacro (robot description, xacro)
@@ -5,10 +5,10 @@
     <xacro:include filename="../models/obstacle.xacro"/>
     <xacro:defineGround
-        vertex="${
+        vertex="${[
             [-10,-10],
             [10,-10],
             [10,10],
             [-10,10]
-        }"
+        ]}"
         origin="${[0,0]}"
     />
@@ -28,4 +28,5 @@
         }"
         initpose="${[0,0,0]}"
+        limit_speed="${[1,0,1,0]}"
     />
     <xacro:defineCargo
