Commit message: Update cargo width and resolution in world.xacro; enhance graph copy assignment operator

File: src/uvs_mapserver/world/jxl3028.world.xacro (robot description, xacro)
@@ -7,5 +7,5 @@
     <!-- 车宽0.238 长 0.34 -->
     <xacro:property name="block_w" value="0.58"/>
-    <xacro:property name="cargo_w" value="0.455"/>
+    <xacro:property name="cargo_w" value="1"/>
     <xacro:macro name="putDefaultCargo" params="name initpose">
         <xacro:defineCargo
@@ -39,6 +39,6 @@
         ]}"
         origin="${[0,0]}"
-        resolutionX="0.025"
-        resolutionY="0.025"
+        resolutionX="0.05"
+        resolutionY="0.05"
     />
     <!-- 长 34.7 宽 23.8 -->

Commit message: Update cargo width in jxl3028 world file and modify CMakeLists to install all library files

File: src/uvs_mapserver/world/jxl3028.world.xacro (robot description, xacro)
@@ -7,5 +7,5 @@
     <!-- 车宽0.238 长 0.34 -->
     <xacro:property name="block_w" value="0.58"/>
-    <xacro:property name="cargo_w" value="1"/>
+    <xacro:property name="cargo_w" value="0.455"/>
     <xacro:macro name="putDefaultCargo" params="name initpose">
         <xacro:defineCargo

Commit message: uvsEmbMaster: send 0 control when quit

File: src/uvs_mapserver/world/jxl3028.world.xacro (robot description, xacro)
@@ -8,4 +8,5 @@
     <xacro:property name="block_w" value="0.58"/>
     <xacro:property name="cargo_w" value="0.455"/>
+    <xacro:property name="obs_w" value="0.455"/>
     <xacro:macro name="putDefaultCargo" params="name initpose">
         <xacro:defineCargo
@@ -24,8 +25,8 @@
     <xacro:macro name="putDefaultObstacle" params="pose">
         <xacro:defineObstacle
-            vertex="${[[-cargo_w/2,-cargo_w/2],
-            [-cargo_w/2,cargo_w/2],
-            [cargo_w/2,cargo_w/2],
-            [cargo_w/2,-cargo_w/2]]}"
+            vertex="${[[-obs_w/2,-obs_w/2],
+            [-obs_w/2,obs_w/2],
+            [obs_w/2,obs_w/2],
+            [obs_w/2,-obs_w/2]]}"
             pose="${pose}"
         />
@@ -57,8 +58,8 @@
         limit_speed="${[1,0,1,0]}"
     />
-    <xacro:putDefaultCargo name="c0" initpose="${[0,0,0]}"/>
     <xacro:putDefaultCargo name="c1" initpose="${[0,0,0]}"/>
     <xacro:putDefaultCargo name="c2" initpose="${[0,0,0]}"/>
     <xacro:putDefaultCargo name="c3" initpose="${[0,0,0]}"/>
+    <xacro:putDefaultCargo name="c4" initpose="${[0,0,0]}"/>
     <xacro:putDefaultObstacle pose="${[0.87,2.61,0]}"/>
     <xacro:putDefaultObstacle pose="${[2.03,0.87,0]}"/>
