Commit message: model in progress

File: src/uvs_gzplugins/worlds/models/Fence/model.xacro (robot description, xacro)
@@ -1,5 +1,74 @@
 <world xmlns:xacro="http://wiki.ros.org/xacro">
 <xacro:property name="wall_thick" value="0.005" />
-<xacro:macro name="putDefaultFence" params="">
+<xacro:property name="wall_height" value="0.515" />
+<xacro:macro name="putDefaultFence" params="name pose wall_len">
+    <model name="${name}">
+        <pose>${pose[0]} ${pose[1]} ${wall_height/2} 0 0 ${pose[2]}</pose>
+        <scale>1 1 1</scale>
+        <static>1</static>
+        <link name='link_0'>
+            <visual name='visual'>
+                <pose>0 0 0 0 -0 0</pose>
+                <geometry>
+                    <box>
+                        <size>${wall_thick} ${wall_len} ${wall_height}</size>
+                    </box>
+                </geometry>
+                <material>
+                    <script>
+                        <uri>file://$(find uvs_gzplugins)/worlds/models/Fence/materials/fence.material</uri>
+                        <name>Uvs/fence</name>
+                    </script>
+                </material>
+            </visual>
+            <collision name='collision'>
+                <pose>0 0 0 0 -0 0</pose>
+                <geometry>
+                    <box>
+                        <size>${wall_thick} ${wall_len} ${wall_height}</size>
+                    </box>
+                </geometry>
+            </collision>
+        </link>
+    </model>
+</xacro:macro>
+<xacro:property name="PI" value="3.14159265359" />
+<xacro:macro name="putSquareFence" params="name ld xlen ylen">
+    <xacro:putDefaultFence
+        name="${name}_1"
+        pose="${[
+            ld[0] - wall_thick/2,
+            ld[1] + ylen/2,
+            0
+        ]}"
+        wall_len="${ylen}"
+    />
+    <xacro:putDefaultFence
+        name="${name}_2"
+        pose="${[
+            ld[0] + xlen + wall_thick/2,
+            ld[1] + ylen/2,
+            0
+        ]}"
+        wall_len="${ylen}"
+    />
+    <xacro:putDefaultFence
+        name="${name}_3"
+        pose="${[
+            ld[0] + xlen/2,
+            ld[1] - wall_thick/2,
+            PI/2
+        ]}"
+        wall_len="${xlen}"
+    />
+    <xacro:putDefaultFence
+        name="${name}_4"
+        pose="${[
+            ld[0] + xlen/2,
+            ld[1] + ylen + wall_thick/2,
+            PI/2
+        ]}"
+        wall_len="${xlen}"
+    />
 </xacro:macro>
 </world>

File: src/uvs_gzplugins/worlds/models/FloorMats/model.xacro (robot description, xacro)
@@ -48,5 +48,5 @@
                 ld_pose[2]
             ]}"
-            color_id="${(lr+ud)%2}"
+            color_id="${(lr+ud+1)%2}"
         />
         <xacro:putMatMatrixLoopUD lr="${lr}" ud="${ud-1}" ld_pose="${ld_pose}"/>
@@ -62,5 +62,5 @@
     <xacro:property name="lr" value="${left+right}"/>
     <xacro:property name="ud" value="${up+down}"/>
-    <xacro:property name="ld_pose" value="${[-block_width*(left-0.5),-block_width*(down-0.5),0]}"/>
+    <xacro:property name="ld_pose" value="${[-block_width*(left+0.5),-block_width*(down+0.5),0]}"/>
     <xacro:putMatMatrixLoopLR lr="${lr}" ud="${ud}" ld_pose="${ld_pose}"/>
 </xacro:macro>

File: src/uvs_gzplugins/worlds/uvs_gazebo.world.xacro (robot description, xacro)
@@ -2,4 +2,7 @@
     <world name='default' xmlns:xacro="http://wiki.ros.org/xacro">
         <xacro:include filename="models/FloorMats/model.xacro" />
+        <xacro:include filename="models/Fence/model.xacro" />
+        <xacro:include filename="models/StaticObstacle/model.xacro" />
+        <xacro:include filename="models/DynamicObstacle/model.xacro" />
         <scene>
             <ambient>0.4 0.4 0.4 1</ambient>
@@ -12,5 +15,36 @@
             <direction>-1 -1 -1</direction>
         </light>
-        <xacro:putMatMatrix left="10" right="10" up="10" down="10" />
+        <xacro:putMatMatrix left="6" right="5" up="8" down="7" />
+        <xacro:putSquareFence name="fence" ld="${[-3.48,-4.06,0]}" xlen="6.38" ylen="8.7" />
+        <xacro:putObstacleList prefix="obstacle" obstacle_list="${[
+            [0.87,2.61,0],
+            [2.03,0.87,0],
+            [-0.29,0.87,0],
+            [-0.29,1.45,0],
+            [-0.29,2.03,0],
+            [-0.29,3.19,0],
+            [-0.29,3.77,0],
+            [-0.29,4.35,0],
+            [-0.87,0.87,0],
+            [-1.45,0.87,0],
+            [-2.03,0.87,0],
+            [-2.61,0.87,0],
+            [-3.19,0.87,0],
+            [-0.29,-0.29,0],
+            [0.29,-0.29,0],
+            [0.87,-0.29,0],
+            [2.03,-0.29,0],
+            [2.61,-0.29,0],
+            [-0.87,-0.87,0],
+            [-1.45,-0.87,0],
+            [-2.61,-0.87,0],
+            [-3.19,-1.45,0]
+        ]}" />
+        <xacro:putCargoList name_list="${['c1','c2','c3','c4']}" initpose_list="${[
+            [-2.0, -0.864, 0.0],
+            [-0.258, 0.249, 0.0],
+            [1.52, -0.316, 0.0],
+            [-0.274, 2.59, 0.0]
+        ]}" />
     </world>
 </sdf>
