Commit message: arm control and emag control success need to be improved

File: src/uvs_gzplugins/worlds/models/Agent/model.xacro (robot description, xacro)
@@ -34,4 +34,12 @@
                     <mesh><uri>file://$(find uvs_gzplugins)/worlds/models/Agent/meshes/base_link.STL</uri></mesh>
                 </geometry>
+                <surface>
+                    <friction>
+                        <ode>
+                            <mu>0.5</mu>
+                            <mu2>0.5</mu2>
+                        </ode>
+                    </friction>
+                </surface>
             </collision>
         </link>
@@ -88,9 +96,9 @@
         </joint>
         <link name="arm">
-            <pose>0.12925 0 -0.014083 -0.7854 0 -1.5708</pose>
+            <pose relative_to="base_link">0.12925 0 -0.014083 -0.7854 0 -1.5708</pose>
             <inertial>
                 <pose>-0.006174 8.44369E-05 0.0132 0 0 0</pose>
                 <mass> 0.067681113134478 </mass>
-                <inertia>
+                <!-- <inertia>
                         <ixx>2.68497509518873E-05</ixx>
                         <ixy>-3.33020165981552E-06</ixy>
@@ -99,5 +107,5 @@
                         <iyz>-4.72072757937217E-06</iyz>
                         <izz>4.4994530861743E-05</izz>
-                </inertia>
+                </inertia> -->
             </inertial>
             <visual name="visual">
@@ -123,5 +131,5 @@
             <child> arm </child>
             <axis><xyz> 0 0 0</xyz> </axis>
-            <pose>0.12925 0 -0.014083 -0.7854 0 -1.5708</pose>
+            <!-- <pose>0.12925 0 -0.014083 -0.7854 0 -1.5708</pose> -->
         </joint>
         <link name="arm_link1">
@@ -130,5 +138,5 @@
                 <pose>-0.00227 0.024777 0.000485 0 1.5708 0</pose>
                 <mass> 0.0315348657457593 </mass>
-                <inertia>
+                <!-- <inertia>
                         <ixx>2.62365924906028E-05</ixx>
                         <ixy>-8.71620806198248E-07</ixy>
@@ -137,5 +145,5 @@
                         <iyz>1.32494709462361E-07</iyz>
                         <izz>2.43479091390021E-05</izz>
-                </inertia>
+                </inertia> -->
             </inertial>
             <visual name="visual">
@@ -166,5 +174,5 @@
                     <lower>-3.927</lower>
                     <upper>0</upper>
-                    <effort>100</effort>
+                    <!-- <effort>100</effort> -->
                     <velocity>1</velocity>
                 </limit>
@@ -177,5 +185,5 @@
                 <pose>-0.012 0.04428 -0.00083 0 0 0</pose>
                 <mass> 0.064068284960248 </mass>
-                <inertia>
+                <!-- <inertia>
                         <ixx>5.32496834034383E-05</ixx>
                         <ixy>1.14801087297394E-05</ixy>
@@ -184,5 +192,5 @@
                         <iyz>1.57043385958373E-06</iyz>
                         <izz>5.71389111747307E-05</izz>
-                </inertia>
+                </inertia> -->
             </inertial>
             <visual name="visual">
@@ -213,5 +221,5 @@
                     <lower>-0.2617</lower>
                     <upper>3.926875</upper>
-                    <effort>100</effort>
+                    <!-- <effort>100</effort> -->
                     <velocity>1</velocity>
                 </limit>
@@ -440,4 +448,21 @@
             <mimic joint="left_joint2"><multiplier>-1</multiplier></mimic>
         </joint> -->
+        <plugin name="uvs_gzplugins_chassis" filename="libgz_ros_simchassis.so">
+            <status_topic>uvs_emb_status</status_topic>
+            <arm_topic>uvs_emb_arm</arm_topic>
+            <emag_topic>uvs_emb_emag</emag_topic>
+            <kinetics_topic>uvs_emb_kinetics</kinetics_topic>
+            <status_pub_period>0.05</status_pub_period>
+            <limit_velocity>0.5</limit_velocity>
+            <limit_anglevelocity>${PI}</limit_anglevelocity>
+            <wheel_separation>0.238</wheel_separation>
+            <arm_base_joint_name>arm_joint1</arm_base_joint_name>
+            <arm_arm_joint_name>arm_joint2</arm_arm_joint_name>
+            <emag_link_name>arm_link2</emag_link_name>
+            <model>c1</model>
+            <model>c2</model>
+            <model>c3</model>
+            <model>c4</model>
+        </plugin>
     </model>
 </xacro:macro>

File: src/uvs_gzplugins/worlds/models/DynamicObstacle/model.xacro (robot description, xacro)
@@ -9,4 +9,15 @@
         <static>0</static>
         <link name='link_0'>
+            <inertial>
+                <mass> 0.06 </mass>
+                <inertia>
+                        <ixx>0</ixx>
+                        <ixy>0</ixy>
+                        <ixz>0</ixz>
+                        <iyy>0</iyy>
+                        <iyz>0</iyz>
+                        <izz>0</izz>
+                </inertia>
+            </inertial>
             <visual name='visual'>
                 <pose>0 0 0 0 -0 0</pose>
@@ -30,4 +41,12 @@
                     </box>
                 </geometry>
+                <surface>
+                    <friction>
+                        <ode>
+                            <mu>0.1</mu>
+                            <mu2>0.1</mu2>
+                        </ode>
+                    </friction>
+                </surface>
             </collision>
         </link>
@@ -48,4 +67,12 @@
                     </sphere>
                 </geometry>
+                <surface>
+                    <friction>
+                        <ode>
+                            <mu>0.02</mu>
+                            <mu2>0.01</mu2>
+                        </ode>
+                    </friction>
+                </surface>
             </collision>
         </link>
@@ -66,4 +93,12 @@
                     </sphere>
                 </geometry>
+                <surface>
+                    <friction>
+                        <ode>
+                            <mu>0.02</mu>
+                            <mu2>0.01</mu2>
+                        </ode>
+                    </friction>
+                </surface>
             </collision>
         </link>
@@ -84,4 +119,12 @@
                     </sphere>
                 </geometry>
+                <surface>
+                    <friction>
+                        <ode>
+                            <mu>0.02</mu>
+                            <mu2>0.01</mu2>
+                        </ode>
+                    </friction>
+                </surface>
             </collision>
         </link>
@@ -102,4 +145,12 @@
                     </sphere>
                 </geometry>
+                <surface>
+                    <friction>
+                        <ode>
+                            <mu>0.02</mu>
+                            <mu2>0.01</mu2>
+                        </ode>
+                    </friction>
+                </surface>
             </collision>
         </link>

File: src/uvs_gzplugins/worlds/models/FloorMats/model.xacro (robot description, xacro)
@@ -35,4 +35,12 @@
                     </box>
                 </geometry>
+                <surface>
+                    <friction>
+                        <ode>
+                            <mu>0.1</mu>
+                            <mu2>0.1</mu2>
+                        </ode>
+                    </friction>
+                </surface>
             </collision>
         </link>

File: src/uvs_gzplugins/worlds/uvs_gazebo.world.xacro (robot description, xacro)
@@ -49,4 +49,13 @@
         ]}" />
         <xacro:putAgent name="uv05" pose="${[-1.5,-1.5,0.1]}" />
+        <plugin name="uvs_gzplugins_optitrack" filename="libgz_ros_simoptitrack.so">
+            <topic>uvs_opt_pose_list</topic>
+            <publish_period>0.01</publish_period>
+            <model>uv05</model>
+            <model>c1</model>
+            <model>c2</model>
+            <model>c3</model>
+            <model>c4</model>
+        </plugin>
     </world>
 </sdf>
