Commit message: all model finished

File: src/uvs_gzplugins/worlds/models/DynamicObstacle/model.xacro (robot description, xacro)
@@ -2,5 +2,5 @@
 <xacro:property name="cargo_width" value="0.41"/>
 <xacro:property name="cargo_height" value="0.31"/>
-<xacro:property name="cargo_wheel_radius" value="0.03"/>
+<xacro:property name="cargo_wheel_radius" value="0.02"/>
 <xacro:macro name="putDefaultCargo" params="name initpose">
     <model name="${name}">

File: src/uvs_gzplugins/worlds/uvs_gazebo.world.xacro (robot description, xacro)
@@ -5,4 +5,5 @@
         <xacro:include filename="models/StaticObstacle/model.xacro" />
         <xacro:include filename="models/DynamicObstacle/model.xacro" />
+        <xacro:include filename="models/Agent/model.xacro" />
         <scene>
             <ambient>0.4 0.4 0.4 1</ambient>
@@ -47,4 +48,5 @@
             [-0.274, 2.59, 0.0]
         ]}" />
+        <xacro:putAgent name="uv05" pose="${[-1.5,-1.5,0.1]}" />
     </world>
 </sdf>

Commit message: Refactor callback functions and update dynamic obstacle model properties for improved simulation accuracy

File: src/uvs_gzplugins/worlds/models/DynamicObstacle/model.xacro (robot description, xacro)
@@ -1,5 +1,6 @@
 <world xmlns:xacro="http://wiki.ros.org/xacro">
 <xacro:property name="cargo_width" value="0.41"/>
-<xacro:property name="cargo_height" value="0.31"/>
+<!-- <xacro:property name="cargo_height" value="0.31"/> -->
+<xacro:property name="cargo_height" value="0.41"/>
 <xacro:property name="cargo_wheel_radius" value="0.02"/>
 <xacro:macro name="putDefaultCargo" params="name initpose">
@@ -12,10 +13,10 @@
                 <mass> 0.06 </mass>
                 <inertia>
-                        <ixx>0</ixx>
-                        <ixy>0</ixy>
-                        <ixz>0</ixz>
-                        <iyy>0</iyy>
-                        <iyz>0</iyz>
-                        <izz>0</izz>
+                        <ixx>0.001681</ixx>
+                        <ixy>0</ixy>
+                        <ixz>0</ixz>
+                        <iyy>0.001681</iyy>
+                        <iyz>0</iyz>
+                        <izz>0.001681</izz>
                 </inertia>
             </inertial>
@@ -51,5 +52,16 @@
             </collision>
         </link>
-        <link name='link_1'>
+        <!-- <link name='link_1'>
+            <inertial>
+                <mass> 0.1 </mass>
+                <inertia>
+                        <ixx>0</ixx>
+                        <ixy>0</ixy>
+                        <ixz>0</ixz>
+                        <iyy>0</iyy>
+                        <iyz>0</iyz>
+                        <izz>0</izz>
+                </inertia>
+            </inertial>
             <visual name='visual'>
                 <pose>${cargo_width/2} ${cargo_width/2} ${-cargo_height/2} 0 -0 0</pose>
@@ -70,6 +82,6 @@
                     <friction>
                         <ode>
-                            <mu>0.2</mu>
-                            <mu2>0.1</mu2>
+                            <mu>1</mu>
+                            <mu2>1</mu2>
                         </ode>
                     </friction>
@@ -78,4 +90,15 @@
         </link>
         <link name='link_2'>
+            <inertial>
+                <mass> 0.1 </mass>
+                <inertia>
+                        <ixx>0</ixx>
+                        <ixy>0</ixy>
+                        <ixz>0</ixz>
+                        <iyy>0</iyy>
+                        <iyz>0</iyz>
+                        <izz>0</izz>
+                </inertia>
+            </inertial>
             <visual name='visual'>
                 <pose>${cargo_width/2} ${-cargo_width/2} ${-cargo_height/2} 0 -0 0</pose>
@@ -96,6 +119,6 @@
                     <friction>
                         <ode>
-                            <mu>0.02</mu>
-                            <mu2>0.01</mu2>
+                            <mu>1</mu>
+                            <mu2>1</mu2>
                         </ode>
                     </friction>
@@ -104,4 +127,15 @@
         </link>
         <link name='link_3'>
+            <inertial>
+                <mass> 0.1 </mass>
+                <inertia>
+                        <ixx>0</ixx>
+                        <ixy>0</ixy>
+                        <ixz>0</ixz>
+                        <iyy>0</iyy>
+                        <iyz>0</iyz>
+                        <izz>0</izz>
+                </inertia>
+            </inertial>
             <visual name='visual'>
                 <pose>${-cargo_width/2} ${-cargo_width/2} ${-cargo_height/2} 0 -0 0</pose>
@@ -122,6 +156,6 @@
                     <friction>
                         <ode>
-                            <mu>0.02</mu>
-                            <mu2>0.01</mu2>
+                            <mu>1</mu>
+                            <mu2>1</mu2>
                         </ode>
                     </friction>
@@ -130,4 +164,15 @@
         </link>
         <link name='link_4'>
+            <inertial>
+                <mass> 0.1 </mass>
+                <inertia>
+                        <ixx>0</ixx>
+                        <ixy>0</ixy>
+                        <ixz>0</ixz>
+                        <iyy>0</iyy>
+                        <iyz>0</iyz>
+                        <izz>0</izz>
+                </inertia>
+            </inertial>
             <visual name='visual'>
                 <pose>${-cargo_width/2} ${cargo_width/2} ${-cargo_height/2} 0 -0 0</pose>
@@ -148,6 +193,6 @@
                     <friction>
                         <ode>
-                            <mu>0.02</mu>
-                            <mu2>0.01</mu2>
+                            <mu>1</mu>
+                            <mu2>1</mu2>
                         </ode>
                     </friction>
@@ -174,5 +219,5 @@
             <child>link_4</child>
             <pose>0 0 0 0 0 0</pose>
-        </joint>
+        </joint> -->
     </model>
 </xacro:macro>
